File: hw/controller/dvernik.kicad_pcb (KiCad board)
At the start: 2 copper layers, 100 x 100 mm, 87 parts, among them P101 WAGO233, P102 CONN_01X06, P103 CONN_01X02, P201 WAGO255, P202 WAGO255, P401 WAGO255, P402 Wago_233-502, P403 Wago_233-502, Q201 2N7002K, Q401 IRFU9024, Q402 IRLML6402, U101 A25L40P, U102 EK-TM4C123GXL, U103 Itead_HC-05, U104 LP2992AIM5-3.3CT-ND, U201 JQX-14FC22CS8-5.0, U202 Cosmo_1010-817, U401 Mini-360, U403 ROE-0505S, U404 HCPL-0601-500E, U405 HCPL-0601-500E, U406 Cosmo_1010-817, U407 SN75176BDR

Commit message: Slight improvements to hardware design
Parts:
- added C401: Jamicon_220uF_25V, th-normal:C_Radial_D8_L11.5_P3.5, F.Cu at (55.2, 112.1)
- added C412: C, smd-handsolder:C_1206_HandSoldering, B.Cu at (61.0, 109.2)
- added U402: Mini-360, th-normal:DcDc_MH_MINI_360, F.Cu at (100.3, 99.1)
- moved C403 54.0 mm to (99.1, 76.2), turned to 270 degrees
- moved C405 47.4 mm to (102.9, 104.1), turned to 270 degrees
- moved REF** 26.5 mm to (91.4, 74.9)
Connections:
- Q401 pad 4: +12V -> Net-(C401-Pad1)
- U401 pad 1: +12V -> Net-(C401-Pad1)
Routing:
- net Net-(C401-Pad1): track 0.00 -> 63.3 mm, vias 0 -> 2
- net +12V: track 133.5 -> 86.0 mm, vias 4 -> 2
- net GND: track 564.1 -> 582.9 mm
- net +5V: track 280.8 -> 281.3 mm
Other:
- board text added: "5V | G"
- board text added: "GND ~12V"
- board text removed: "5V / G"
- board text removed: "GND 12V"
