File: hw/reader/reader.kicad_pcb (KiCad board)
At the start: 2 copper layers, 50 x 50 mm, 40 parts, among them P101 Wago_233-502, P102 Wago_233-502, P103 CONN_02X05, P104 JST, P105 CONN_01X08, Q101 MMBT2222A, Q102 MMBT2222A, U101 LP2992AIM5-3.3CT-ND, U102 SN75176BDR, U103 MKE04P24M48SF0, X101 CRYSTAL

Commit message: Slight improvements to hardware design
Parts:
- moved C110 4.00 mm to (64.0, 61.4)
- moved R110 1.11 mm to (65.2, 58.9)
- moved REF** 1.00 mm to (95.0, 56.0)
- moved REF** 1.00 mm to (55.0, 56.0)
Connections:
- U103 pad 11: Net-(U103-Pad11) -> /IRQ
Routing:
- net /IRQ: track 0.00 -> 15.5 mm, vias 0 -> 1
- net +3V3: track 156.0 -> 154.5 mm
- net /~RE_RESET: track 13.0 -> 11.8 mm
