File: hw/reader/reader.sch (KiCad schematic (older format))
At the start: 35 parts, among them P101 Wago_233-502, P102 Wago_233-502, P103 CONN_02X05, P104 JST, P105 CONN_01X08, Q101 MMBT2222A, Q102 MMBT2222A, U101 LP2992AIM5-3.3CT-ND, U102 SN75176BDR, U103 MKE04P24M48SF0, X101 CRYSTAL

Commit message: Slight improvements to hardware design
Connections:
- wire segments 109 -> 110
- no-connect marks 7 -> 5
Changed lines of the file:
@@
 Text Label 6900 3250 0    60   ~ 0
 ~RE_RESET
-NoConn ~ 6850 3350
 Text Label 10100 3750 2    60   ~ 0
 ~RE_RESET
@@
 	1    0    0    -1
 $EndComp
-NoConn ~ 9600 3950
 $Comp
 L PWR_FLAG #FLG037
@@
 Text Label 2200 6700 0    60   ~ 0
 485B
+Wire Wire Line
+	6850 3350 7350 3350
+Text Label 6900 3350 0    60   ~ 0
+IRQ
 $EndSCHEMATC
