File: controller/hw/dvernik.kicad_pcb (KiCad board)
At the start: 2 copper layers, 100 x 100 mm, 90 parts, among them P101 WAGO233, P102 CONN_01X06, P103 CONN_01X02, P201 WAGO255, P202 WAGO255, P401 WAGO255, P402 Wago_233-502, P403 Wago_233-502, Q201 2N7002K, Q401 IRFU9024, Q402 IRLML6402, U101 A25L40P, U102 EK-TM4C123GXL, U103 Itead_HC-05, U104 LP2992AIM5-3.3CT-ND, U201 JQX-14FC22CS8-5.0, U202 Cosmo_1010-817, U401 Mini-360, U402 Mini-360, U403 ROE-0505S, U404 HCPL-0601-500E, U405 HCPL-0601-500E, U406 Cosmo_1010-817, U407 SN75176BDR

Commit message: Restructure files and small updates
Other:
- board text added: "CHARGE +BATT CURRENT1 CURRENT2 VCC GND"
Changed lines of the file:
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@@
-(kicad_pcb (version 20170123) (host pcbnew "(2017-05-12 revision b823d0b)-master")
+(kicad_pcb (version 20170123) (host pcbnew "(2017-05-18 revision 2a3a699)-master")
   (general
     (links 201)
-    (no_connects 3)
+    (no_connects 0)
     (area 46.361476 47.2485 154.688524 175.589001)
     (thickness 1.6)
-    (drawings 20)
+    (drawings 21)
     (tracks 789)
     (zones 0)
@@
   )
   (setup
-    (last_trace_width 1.27)
+    (last_trace_width 0.508)
     (user_trace_width 0.508)
     (user_trace_width 1.016)
@@
       (drillshape 0)
       (scaleselection 1)
-      (outputdirectory dirtypcb/))
+      (outputdirectory seedstudio/))
   )
   (net 0 "")
@@
     )
   )
+  (gr_text "CHARGE\n+BATT\nCURRENT1\nCURRENT2\nVCC\nGND" (at 94.615 118.745) (layer F.SilkS)
+    (effects (font (size 1 1) (thickness 0.15)) (justify left))
+  )
   (gr_text "GND\n~12V" (at 50.8 80.645) (layer F.SilkS)
