File: controller/hw/door.sch (KiCad schematic (older format))
At the start: 14 parts, among them P201 WAGO255, P202 WAGO255, Q201 2N7002K, U201 JQX-14FC22CS8-5.0, U202 Cosmo_1010-817

Commit message: Compilability using embc lm4f, fixes to TX_EN switching
Parts:
- C201: symbol Jamicon_220uF_16V_TKP -> capacitors:Jamicon_220uF_16V_TKP
- D201: symbol SK110 -> simple:SK110
- D202, D203, D204, D205: symbol SD103A -> simple:SD103A
- F201: symbol FUSE -> templates:FUSE
- P201: symbol CONN_01X02 -> connectors:CONN_01X02
- P202: symbol CONN_01X03 -> connectors:CONN_01X03
- Q201: symbol 2N7002K -> transistors:2N7002K
- R201, R202: symbol R -> simple:R
- U201: symbol JQX-14FC22CS8-5.0 -> relay:JQX-14FC22CS8-5.0
- U202: symbol Cosmo_1010-817 -> opto:Cosmo_1010-817
Changed lines of the file:
@@
-EESchema Schematic File Version 2
-LIBS:74xx
-LIBS:boards
-LIBS:buttons
-LIBS:capacitors
-LIBS:connectors
-LIBS:cpu
-LIBS:discrete
-LIBS:drivers
-LIBS:ic
-LIBS:mspower
-LIBS:opto
-LIBS:passives
-LIBS:power
-LIBS:relay
-LIBS:rf
-LIBS:simple
-LIBS:transistors
-LIBS:templates
+EESchema Schematic File Version 4
 LIBS:dvernik-cache
 EELAYER 26 0
@@
 $EndDescr
 $Comp
-L JQX-14FC22CS8-5.0 U201
+L relay:JQX-14FC22CS8-5.0 U201
 U 1 1 58FE8C56
 P 5700 3300
@@
 $EndComp
 $Comp
-L 2N7002K Q201
+L transistors:2N7002K Q201
 U 1 1 58FE8C63
 P 5300 4100
@@
 $EndComp
 $Comp
-L SK110 D201
+L simple:SK110 D201
 U 1 1 58FE8C6A
 P 4900 3300
@@
 $EndComp
 $Comp
-L R R201
+L simple:R R201
 U 1 1 58FE8C83
 P 4650 4300
@@
 TODO - is the mosfet strong enough?\n24mA at Vgs = 3.3V; Vds = 5V within specs\n(Rdson cca 5 ohm)
 $Comp
-L Jamicon_220uF_16V_TKP C201
+L capacitors:Jamicon_220uF_16V_TKP C201
 U 1 1 58FE8C97
 P 4350 3000
@@
 OPEN
 $Comp
-L CONN_01X02 P201
+L connectors:CONN_01X02 P201
 U 1 1 58FE8E7A
 P 6350 2300
@@
 Log. high triggers the relay\nand opens the door
 $Comp
-L CONN_01X03 P202
+L connectors:CONN_01X03 P202
 U 1 1 58FEE200
 P 8600 4200
@@
 The replacement buzzer power,\npolarity normally does not matter
 $Comp
-L SD103A D205
+L simple:SD103A D205
 U 1 1 5916DE27
 P 8000 2600
@@
 $EndComp
 $Comp
-L SD103A D202
+L simple:SD103A D202
 U 1 1 5916DE99
 P 7500 1950
@@
 $EndComp
 $Comp
-L SD103A D204
+L simple:SD103A D204
 U 1 1 5916DEC5
 P 8000 1950
@@
 $EndComp
 $Comp
-L SD103A D203
+L simple:SD103A D203
 U 1 1 5916DEF3
 P 7500 2600
@@
 $EndComp
 $Comp
-L Cosmo_1010-817 U202
+L opto:Cosmo_1010-817 U202
 U 1 1 5916DFF3
 P 9800 3100
@@
 $EndComp
 $Comp
-L R R202
+L simple:R R202
 U 1 1 5916E13C
 P 9250 3200
@@
 	4150 2550 5400 2550
 $Comp
-L FUSE F201
+L templates:FUSE F201
 U 1 1 591740C4
 P 7050 5050
