File: reader/hw/reader.kicad_pcb (KiCad board)
At the start: 2 copper layers, 50 x 50 mm, 40 parts, among them P101 Wago_233-502, P102 Wago_233-502, P103 CONN_02X05, P104 JST, P105 CONN_01X08, Q101 MMBT2222A, Q102 MMBT2222A, U101 LP2992AIM5-3.3CT-ND, U102 SN75176BDR, U103 MKE04P24M48SF0, X101 CRYSTAL

Commit message: Restructure files and small updates
Parts:
- added R112: R, smd-handsolder:R_1206_HandSoldering, F.Cu at (80.5, 63.3)
Routing:
- net /CPU_TX: track 16.7 -> 21.3 mm, vias 0 -> 1
- net +3V3: track 154.5 -> 157.0 mm
- net GND: track 269.5 -> 271.6 mm
Changed lines of the file:
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@@
 (kicad_pcb (version 20170123) (host pcbnew "(2017-05-18 revision 2a3a699)-master")
   (general
-    (links 83)
-    (no_connects 1)
+    (links 85)
+    (no_connects 2)
     (area 46.704486 47.086866 102.594086 110.100001)
     (thickness 1.6)
     (drawings 18)
-    (tracks 327)
+    (tracks 334)
     (zones 0)
-    (modules 40)
+    (modules 41)
     (nets 34)
   )
@@
     (visible_elements FFFFFF7F)
     (pcbplotparams
-      (layerselection 0x00030_ffffffff)
+      (layerselection 0x010f0_ffffffff)
       (usegerberextensions false)
       (excludeedgelayer true)
@@
       (outputformat 1)
       (mirror false)
-      (drillshape 1)
+      (drillshape 0)
       (scaleselection 1)
-      (outputdirectory ""))
+      (outputdirectory seedstudio/))
   )
   (net 0 "")
@@
       (net 6 "Net-(C108-Pad1)"))
   )
+  (module smd-handsolder:R_1206_HandSoldering (layer F.Cu)
+    (at 80.48 63.335 90)
+    (descr "Resistor SMD 1206, hand soldering")
+    (tags "resistor 1206")
+    (attr smd)
+    (fp_text reference R112 (at 2.54 3.175 180) (layer F.SilkS)
+      (effects (font (size 1 1) (thickness 0.15)))
+    )
+    (fp_text value R (at 0 2.3 90) (layer F.Fab)
+      (effects (font (size 1 1) (thickness 0.15)))
+    )
+    (fp_line (start -3.3 -1.2) (end 3.3 -1.2) (layer F.CrtYd) (width 0.05))
+    (fp_line (start -3.3 1.2) (end 3.3 1.2) (layer F.CrtYd) (width 0.05))
+    (fp_line (start -3.3 -1.2) (end -3.3 1.2) (layer F.CrtYd) (width 0.05))
+    (fp_line (start 3.3 -1.2) (end 3.3 1.2) (layer F.CrtYd) (width 0.05))
+    (fp_line (start 1 1.075) (end -1 1.075) (layer F.SilkS) (width 0.15))
+    (fp_line (start -1 -1.075) (end 1 -1.075) (layer F.SilkS) (width 0.15))
+    (pad 1 smd rect (at -2 0 90) (size 2 1.7) (layers F.Cu F.Paste F.Mask)
+      (net 4 +3V3))
+    (pad 2 smd rect (at 2 0 90) (size 2 1.7) (layers F.Cu F.Paste F.Mask)
+      (net 30 /CPU_TX))
+    (model Resistors_SMD.3dshapes/R_1206_HandSoldering.wrl
+      (at (xyz 0 0 0))
+      (scale (xyz 1 1 1))
+      (rotate (xyz 0 0 0))
+    )
+  )
   (gr_text "3.3V\nRESET\nGND\nIRQ\nMISO\nMOSI\nSCK\nCS" (at 83.02 56.985 90) (layer F.SilkS)
     (effects (font (size 1 1) (thickness 0.15)))
@@
   (segment (start 74.86 96.99) (end 77.59 96.99) (width 0.508) (layer B.Cu) (net 2))
   (segment (start 77.59 96.99) (end 77.91 96.67) (width 0.508) (layer B.Cu) (net 2))
+  (segment (start 95.72 61.43) (end 89.37 67.78) (width 0.508) (layer F.Cu) (net 3))
+  (segment (start 89.37 67.78) (end 77.94 67.78) (width 0.508) (layer F.Cu) (net 3))
+  (segment (start 77.94 67.78) (end 75.4 65.24) (width 0.508) (layer F.Cu) (net 3))
   (segment (start 94.45 72.86) (end 94.45 74.13) (width 1.016) (layer F.Cu) (net 3))
   (segment (start 94.45 74.13) (end 91.91 76.67) (width 0.508) (layer F.Cu) (net 3))
@@
   (via (at 89.37 71.59) (size 1.5) (drill 0.8) (layers F.Cu B.Cu) (net 3))
   (segment (start 67.05 87.56) (end 66.51 88.1) (width 0.508) (layer B.Cu) (net 3))
-  (segment (start 95.72 61.43) (end 91.91 65.24) (width 0.508) (layer F.Cu) (net 3))
-  (segment (start 91.91 65.24) (end 75.4 65.24) (width 0.508) (layer F.Cu) (net 3))
   (segment (start 93.72 63.97) (end 93.72 63.43) (width 0.508) (layer B.Cu) (net 3))
   (segment (start 93.72 63.43) (end 95.72 61.43) (width 0.508) (layer B.Cu) (net 3))
@@
   (segment (start 78.48 71.59) (end 77.94 71.05) (width 0.508) (layer B.Cu) (net 3))
   (segment (start 77.94 71.05) (end 77.94 68.29) (width 0.508) (layer B.Cu) (net 3))
+  (segment (start 77.94 62.7) (end 80.48 62.893801) (width 0.508) (layer F.Cu) (net 4))
+  (segment (start 80.48 62.893801) (end 86.807178 62.7) (width 0.508) (layer F.Cu) (net 4))
+  (segment (start 80.48 65.335) (end 80.48 62.893801) (width 0.508) (layer F.Cu) (net 4))
   (segment (start 63.97 61.43) (end 61.43 61.43) (width 0.508) (layer B.Cu) (net 4))
   (segment (start 61.43 61.43) (end 61.43 56.985) (width 0.508) (layer B.Cu) (net 4))
@@
   (segment (start 90.64 57.62) (end 90.1 57.62) (width 0.508) (layer B.Cu) (net 4))
   (segment (start 90.1 57.62) (end 88.83 56.35) (width 0.508) (layer B.Cu) (net 4))
-  (segment (start 77.94 62.7) (end 86.807178 62.7) (width 0.508) (layer F.Cu) (net 4))
   (segment (start 86.807178 62.7) (end 90.64 58.867178) (width 0.508) (layer F.Cu) (net 4))
   (segment (start 90.64 58.867178) (end 90.64 57.62) (width 0.508) (layer F.Cu) (net 4))
@@
   (segment (start 79.21 58.89) (end 79.21 60.373) (width 0.508) (layer B.Cu) (net 29))
   (segment (start 79.21 60.373) (end 81.537 62.7) (width 0.508) (layer B.Cu) (net 29))
+  (segment (start 77.94 60.795) (end 77.94 58.89) (width 0.508) (layer B.Cu) (net 30))
+  (segment (start 80.48 61.335) (end 78.48 61.335) (width 0.508) (layer F.Cu) (net 30))
+  (segment (start 78.48 61.335) (end 77.94 60.795) (width 0.508) (layer F.Cu) (net 30))
+  (via (at 77.94 60.795) (size 1.5) (drill 0.8) (layers F.Cu B.Cu) (net 30))
   (segment (start 77.94 58.89) (end 77.94 60.373) (width 0.508) (layer B.Cu) (net 30))
   (segment (start 77.94 60.373) (end 83.820801 66.253801) (width 0.508) (layer B.Cu) (net 30))
